File: BoardFiles/AQM/AQM.kicad_pcb (KiCad board)
At the start: 4 copper layers, 60.2 x 50.2 mm, 66 parts, among them J1 Conn_01x04, J2 Conn_01x04, J3 Conn_01x04, J4 Conn_01x04, J5 Conn_01x04, J6 Conn_01x03, J7 LED, J8 USER BUTTON, Q1 BSS138, SW1 SW_Push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

Commit message: Fixing pin swap
Parts:
- R8: value 1k -> 100
- moved C7 3.71 mm to (162.5, 125.8), turned to 0 degrees
- moved C9 3.71 mm to (162.6, 127.8), turned to 0 degrees
- moved C12 3.40 mm to (137.2, 127.8), turned to 0 degrees
- moved C15 3.40 mm to (137.2, 125.8), turned to 0 degrees
- moved C11 3.20 mm to (128.5, 127.8), turned to 0 degrees
- moved C14 3.20 mm to (128.5, 125.8), turned to 0 degrees
- moved C13 3.20 mm to (153.7, 127.8), turned to 0 degrees
- moved C16 3.20 mm to (153.7, 125.8), turned to 0 degrees
- moved C10 2.79 mm to (144.8, 127.8), turned to 0 degrees
- moved C8 2.79 mm to (144.8, 125.8), turned to 0 degrees
Connections:
- J1 pad 1: /I2C/I2C.SCL -> GND
- J1 pad 2: /I2C/I2C.SDA -> Net-(C7-Pad1)
- J1 pad 3: Net-(C7-Pad1) -> /I2C/I2C.SDA
- J1 pad 4: GND -> /I2C/I2C.SCL
- J2 pad 1: /I2C/I2C.SCL -> GND
- J2 pad 2: /I2C/I2C.SDA -> Net-(C10-Pad1)
- J2 pad 3: Net-(C10-Pad1) -> /I2C/I2C.SDA
- J2 pad 4: GND -> /I2C/I2C.SCL
- J3 pad 1: /I2C/I2C.SCL -> GND
- J3 pad 2: /I2C/I2C.SDA -> Net-(C11-Pad1)
- J3 pad 3: Net-(C11-Pad1) -> /I2C/I2C.SDA
- J3 pad 4: GND -> /I2C/I2C.SCL
- J4 pad 1: /I2C/I2C.SCL -> GND
- J4 pad 2: /I2C/I2C.SDA -> Net-(C12-Pad1)
- J4 pad 3: Net-(C12-Pad1) -> /I2C/I2C.SDA
- J4 pad 4: GND -> /I2C/I2C.SCL
- J5 pad 1: /I2C/I2C.SCL -> GND
- J5 pad 2: /I2C/I2C.SDA -> Net-(C13-Pad1)
- J5 pad 3: Net-(C13-Pad1) -> /I2C/I2C.SDA
- J5 pad 4: GND -> /I2C/I2C.SCL
Routing:
- net GND: track 13.5 -> 0.00 mm
- net /I2C/I2C.SCL: track 61.7 -> 57.0 mm, vias 5 -> 6
- net Net-(JP3-Pad2): track 2.94 -> 7.34 mm, vias 0 -> 1
- net Net-(C7-Pad1): track 7.06 -> 8.23 mm
- net Net-(C13-Pad1): track 7.44 -> 8.27 mm
